Commit message: urdf

File: assets/SC_ur10e.urdf (robot description, URDF)
Before this commit: robot ur10e, 7 links, 6 joints
Links:
- link base_link: geometry collision box size=1 1 1; collision mesh filename=meshes/ur10e/collision/base.stl
Joints:
- joint elbow_joint: limit lower=-3.14159 upper=3.14159 effort=150.0 velocity=3.14 -> lower=-3.14159 upper=3.14159 effort=150.0 velocity=2.0944
- joint shoulder_lift_joint: limit lower=-6.283185 upper=6.283185 effort=330.0 velocity=3.14 -> lower=-6.283185 upper=6.283185 effort=330.0 velocity=2.0944
- joint shoulder_pan_joint: limit lower=-6.283185 upper=6.283185 effort=330.0 velocity=3.14 -> lower=-6.283185 upper=6.283185 effort=330.0 velocity=2.0944
- joint wrist_1_joint: limit lower=-6.283185 upper=6.283185 effort=54.0 velocity=6.28 -> lower=-6.283185 upper=6.283185 effort=54.0 velocity=3.14159
- joint wrist_2_joint: limit lower=-6.283185 upper=6.283185 effort=54.0 velocity=6.28 -> lower=-6.283185 upper=6.283185 effort=54.0 velocity=3.14159
- joint wrist_3_joint: limit lower=-6.283185 upper=6.283185 effort=54.0 velocity=6.28 -> lower=-6.283185 upper=6.283185 effort=54.0 velocity=3.14159
