Commit message: Add Monte Carlo weight sweep, improve orientation error display
- Add comparing/montecarlo_weights.py: sweep over 125 weight combinations
  with heatmaps (orient error, joint error, joint vel error), Pareto plot,
  and 1D slice plots
- Add comparing/run_ddp.py: standalone DDP runner with euler deg and
  geodesic angle output for direct comparison with heatmap metrics
- Update scenario.py weights: orient=10, joint_vel=100
- Fix URDF shoulder_lift_joint rpy offset

Co-Authored-By: Claude Opus 4.6 <noreply@anthropic.com>

File: assets/SC_ur10e.urdf (robot description, URDF)
Before this commit: robot ur10e, 7 links, 6 joints
Joints:
- joint shoulder_lift_joint: origin xyz=0.0 0.176 0.0 rpy=0.0 1.5708 0.0 -> xyz=0.0 0.176 0.0 rpy=0.0 0.0 0.0
